File: Erweiterungen/Magnetbandanschluss/Magnetbandanschluss.sch (KiCad schematic (older format))
At the start: 22 parts, among them T1 SC307, U16 DL000D, U17 B555D, U18 B761D, X12 Anschluss, X13 DIN-3

Commit message: Magnetbandanschluss (Platine) hinzugefügt, PDFs umbenannt
Parts:
- removed D4: VQA13, symbol RFT_Optoelektronik:VQA13
- removed R12: 220, symbol Device:R
- removed R16: 47k, symbol Device:RTRIM
- removed X12: Anschluss, symbol Connector_Generic:Conn_01x05
- added R16: 47k, Potentiometer_THT:Potentiometer_Piher_PT-10-H01_Horizontal, symbol Device:R_POT_Small
- added TP1: E, Connector_Pin:Pin_D1.0mm_L10.0mm, symbol Connector:TestPoint_Small
- added TP2: A, Connector_Pin:Pin_D1.0mm_L10.0mm, symbol Connector:TestPoint_Small
- added TP3: L, Connector_Pin:Pin_D1.0mm_L10.0mm, symbol Connector:TestPoint_Small
- added TP4: D, Connector_Pin:Pin_D1.0mm_L10.0mm, symbol Connector:TestPoint_Small
- added X1: +5V, Connector_Pin:Pin_D1.0mm_L10.0mm, symbol Connector_Generic:Conn_01x01
- added X12: P3.0, Connector_Pin:Pin_D1.0mm_L10.0mm, symbol Connector_Generic:Conn_01x01
- added X2: P3.7, Connector_Pin:Pin_D1.0mm_L10.0mm, symbol Connector_Generic:Conn_01x01
- added X3: P3.6, Connector_Pin:Pin_D1.0mm_L10.0mm, symbol Connector_Generic:Conn_01x01
- added X4: 00, Connector_Pin:Pin_D1.0mm_L10.0mm, symbol Connector_Generic:Conn_01x01
- C13, C16: footprint (none) -> Capacitor_THT:C_Disc_D3.0mm_W1.6mm_P2.50mm
- C14, C15: footprint (none) -> Capacitor_THT:C_Axial_L3.8mm_D2.6mm_P12.50mm_Horizontal
- C17: footprint (none) -> Capacitor_THT:CP_Radial_D5.0mm_P2.50mm
- C18: footprint (none) -> Capacitor_THT:CP_Radial_D6.3mm_P2.50mm
- R13, R14, R15, R17, R18, R19: footprint (none) -> Resistor_THT:R_Axial_DIN0309_L9.0mm_D3.2mm_P12.70mm_Horizontal
- T1: footprint (none) -> Package_TO_SOT_THT:TO-92L_Inline_Wide
- U16: footprint (none) -> Package_DIP:DIP-14_W7.62mm_Socket
- U17: footprint Package_DIP:DIP-8_W7.62mm -> Package_DIP:DIP-8_W7.62mm_Socket
- U18: footprint Package_DIP:DIP-6_W7.62mm -> Package_DIP:DIP-6_W7.62mm_Socket
Connections:
- net labels removed: L
- wire segments 87 -> 85
