File: Erweiterungen/Tastatur/Tastatur.sch (KiCad schematic (older format))
At the start: 51 parts, among them SW1 CUU/CUD, SW10 9, SW11 0, SW12 CLR, SW13 CUL/CUR, SW14 Q, SW15 W, SW16 E, SW17 R, SW18 T, SW19 Z, SW2 1, SW20 U, SW21 I, SW22 O, SW23 P, SW24 +, SW25 Shift, SW26 A, SW27 S, SW28 D, SW29 F, SW3 2, SW30 G, SW31 H, SW32 J, SW33 K, SW34 L, SW35 *, SW36 -, SW37 Space, SW38 Y, SW39 X, SW4 3, SW40 C, SW41 V, SW42 B, SW43 N, SW44 M, SW45 <, SW46 >, SW47 /, SW48 Enter, SW5 4, SW6 5, SW7 6, SW8 7, SW9 8, U7 MH74154, X11 Tastatur

Commit message: Platine für Tastatur ergänzt
Parts:
- added H1, H2, H3, H4: M3,5, MountingHole:MountingHole_3.5mm, symbol Mechanical:MountingHole
- C12: footprint (none) -> Capacitor_THT:C_Disc_D4.3mm_W1.9mm_P5.00mm
- SW1, SW10, SW11, SW12, SW13, SW14, SW15, SW16, SW17, SW18, SW19, SW2, SW20, SW21, SW22, SW23, SW24, SW25, SW26, SW27, SW28, SW29, SW3, SW30, SW31, SW32, SW33, SW34, SW35, SW36, SW37, SW38, SW39, SW4, SW40, SW41, SW42, SW43, SW44, SW45, SW46, SW47, SW48, SW5, SW6, SW7, SW8, SW9: footprint (none) -> Tiny2k_Bauteile:TSE15_stehend_ohne_Beleuchtung
- U1: renamed from U7; footprint (none) -> Package_DIP:DIP-24_W15.24mm_Socket
- X11: footprint (none) -> Connector_Molex:Molex_SL_171971-0010_1x10_P2.54mm_Vertical
