File: Erweiterungen/Magnetbandinterface_4k-System/Magnetbandinterface_4k-System.sch (KiCad schematic (older format))
At the start: 32 parts, among them T1 SC238, T2 SC238, U17 B555D, U18 B761D, X1 BAS, X12 Anschluss, X13 DIN-3, X2 Video

Commit message: Referenz korrigiert
Other:
- note added: "Quelle: jutecomp2.pdf S. 30"
- note removed: "Quelle: jutecomp1.pdf S. 30"
Changed lines of the file:
@@
 $EndDescr
 Text Notes 9950 7000 0    50   ~ 0
-Quelle: jutecomp1.pdf  S. 30
+Quelle: jutecomp2.pdf  S. 30
 Text Notes 9950 6900 0    50   ~ 0
 Quelle: JU+TE 3/1989, Seite 230-235

Commit message: Platine für Magnetbandinterface 4k-System ergänzt
Parts:
- removed C15: 22nF, Capacitor_THT:C_Disc_D4.3mm_W1.9mm_P5.00mm, symbol Device:C_Small
- removed R15: 3,3k, Resistor_THT:R_Axial_DIN0207_L6.3mm_D2.5mm_P10.16mm_Horizontal, symbol Device:R
- removed R17, R18: 100k, Resistor_THT:R_Axial_DIN0207_L6.3mm_D2.5mm_P10.16mm_Horizontal, symbol Device:R
- removed X1: BAS, symbol Connector_Generic:Conn_01x01
- removed X12: Anschluss, Connector_PinHeader_2.54mm:PinHeader_1x05_P2.54mm_Vertical, symbol Connector_Generic:Conn_01x05
- removed X2: Video, symbol Connector_Generic:Conn_01x01
- added R15: 3,3k, Tiny2k_Bauteile:R_Axial_TGL8728_L5.9mm_D2.4mm_P12.50mm_Horizontal, symbol Device:R_Small
- added R17, R18: 100k, Tiny2k_Bauteile:R_Axial_TGL8728_L5.9mm_D2.4mm_P12.50mm_Horizontal, symbol Device:R_Small
- added TP1: E, TestPoint:TestPoint_Loop_D2.54mm_Drill1.5mm_Beaded, symbol Connector:TestPoint_Small
- added TP10: L, TestPoint:TestPoint_Loop_D2.54mm_Drill1.5mm_Beaded, symbol Connector:TestPoint_Small
- added TP2: 00, TestPoint:TestPoint_Loop_D2.54mm_Drill1.5mm_Beaded, symbol Connector:TestPoint_Small
- added TP3: A, TestPoint:TestPoint_Loop_D2.54mm_Drill1.5mm_Beaded, symbol Connector:TestPoint_Small
- added X4: P3.6, TestPoint:TestPoint_Loop_D2.54mm_Drill1.5mm_Beaded, symbol Connector_Generic:Conn_01x01
- added X5: P3.0, TestPoint:TestPoint_Loop_D2.54mm_Drill1.5mm_Beaded, symbol Connector_Generic:Conn_01x01
- added X6: 00, TestPoint:TestPoint_Loop_D2.54mm_Drill1.5mm_Beaded, symbol Connector_Generic:Conn_01x01
- added X7: BAS, TestPoint:TestPoint_Loop_D2.54mm_Drill1.5mm_Beaded, symbol Connector_Generic:Conn_01x01
- added X8: Video, TestPoint:TestPoint_Loop_D2.54mm_Drill1.5mm_Beaded, symbol Connector_Generic:Conn_01x01
- added X9: 5V, TestPoint:TestPoint_Loop_D2.54mm_Drill1.5mm_Beaded, symbol Connector_Generic:Conn_01x01
- C1: footprint (none) -> Capacitor_THT:CP_Radial_D6.3mm_P2.50mm
- C13: footprint Capacitor_THT:C_Disc_D4.3mm_W1.9mm_P5.00mm -> Capacitor_THT:C_Rect_L9.0mm_W2.5mm_P7.50mm_MKT
- C14: footprint (none) -> Capacitor_THT:C_Rect_L9.0mm_W2.5mm_P7.50mm_MKT
- C2: value 100p -> 100pF; footprint Capacitor_THT:C_Disc_D4.3mm_W1.9mm_P5.00mm -> Capacitor_THT:C_Rect_L9.0mm_W2.5mm_P7.50mm_MKT
- C3: footprint (none) -> Capacitor_THT:C_Disc_D4.3mm_W1.9mm_P5.00mm
- R1, R13, R14, R19, R2, R3, R4, R5, R6, R7, R8: footprint (none) -> Tiny2k_Bauteile:R_Axial_TGL8728_L5.9mm_D2.4mm_P12.50mm_Horizontal
- T1: value SC238 -> SC238d; footprint (none) -> Package_TO_SOT_THT:TO-92_Inline_Wide
- T2: footprint (none) -> Package_TO_SOT_THT:TO-92_Inline_Wide
- U17: footprint Package_DIP:DIP-8_W7.62mm_Socket -> Package_DIP:DIP-8_W7.62mm
- U18: footprint Package_DIP:DIP-6_W7.62mm_Socket -> Package_DIP:DIP-6_W7.62mm
Connections:
- wire segments 91 -> 94
- no-connect marks 4 -> 3
Other:
- moved on the sheet: C1, C16, C2, R1, R4, R5, T2

Commit message: Kommentar ergänzt
Other:
- note added: "bei Schwingneigung 22pF\nzwischen Pin 5 und 6 ergänzen,\ndamit wird U17 im 4k-System entbehrlich,\nstattdessen Brücke zwische Pin 2 und Pin 3"
Changed lines of the file:
@@
 	1    0    0    -1
 $EndComp
+Text Notes 5650 6500 0    50   ~ 0
+bei Schwingneigung 22pF\nzwischen Pin 5 und 6 ergänzen,\ndamit wird U17 im 4k-System entbehrlich,\nstattdessen Brücke zwische Pin 2 und Pin 3
 $EndSCHEMATC
