File: Erweiterungen/Videoerweiterung/Videoerweiterung_Ausgabe.sch (KiCad schematic (older format))
At the start: 51 parts, among them X400 SCART-F

Commit message: Platine für Videomodul ergänzt
Parts:
- removed JP400: HR direkt, Connector_PinHeader_2.54mm:PinHeader_1x02_P2.54mm_Vertical, symbol Device:Jumper_NC_Small
- removed JP401: HR_VCC, Connector_PinHeader_2.54mm:PinHeader_1x02_P2.54mm_Vertical, symbol Device:Jumper_NO_Small
- removed JP402: HR_GND, Connector_PinHeader_2.54mm:PinHeader_1x02_P2.54mm_Vertical, symbol Device:Jumper_NO_Small
- removed R400, R402, R403: 160, Resistor_THT:R_Axial_DIN0207_L6.3mm_D2.5mm_P10.16mm_Horizontal, symbol Device:R_Small
- removed R401: 75, Resistor_THT:R_Axial_DIN0207_L6.3mm_D2.5mm_P10.16mm_Horizontal, symbol Device:R_Small
- removed R404: 51, Resistor_THT:R_Axial_DIN0207_L6.3mm_D2.5mm_P10.16mm_Horizontal, symbol Device:R_Small
- removed R405, R406, R407: 220, Resistor_THT:R_Axial_DIN0207_L6.3mm_D2.5mm_P10.16mm_Horizontal, symbol Device:R_Small
- removed R408: 100, Resistor_THT:R_Axial_DIN0207_L6.3mm_D2.5mm_P10.16mm_Horizontal, symbol Device:R
- removed X400: SCART-F, Connector_PinHeader_2.54mm:PinHeader_1x21_P2.54mm_Vertical, symbol Connector:SCART-F
- added C10, C12, C13, C14, C15, C17, C20, C24, C4, C5, C7, C8, C9: 22nF, Capacitor_THT:C_Disc_D3.0mm_W1.6mm_P2.50mm, symbol Device:C_Small
- added C18: 22nF, Capacitor_THT:C_Disc_D4.3mm_W1.9mm_P5.00mm, symbol Device:C_Small
- added C19, C22, C23, C3: 100nF, Capacitor_THT:C_Disc_D4.3mm_W1.9mm_P5.00mm, symbol Device:C_Small
- added C2: 220µF/16V, Tiny2k_Bauteile:CP_Axial_L25.0mm_D10.0mm_P30.00mm_Horizontal, symbol Device:CP_Small
- added NT1: Net-Tie_2, NetTie:NetTie-2_SMD_Pad0.5mm, symbol Device:Net-Tie_2
- added X400, X405: V, Connector_PinHeader_2.54mm:PinHeader_1x01_P2.54mm_Vertical, symbol Connector_Generic:Conn_01x01
- added X401: B, Connector_PinHeader_2.54mm:PinHeader_1x01_P2.54mm_Vertical, symbol Connector_Generic:Conn_01x01
- added X402: S, Connector_PinHeader_2.54mm:PinHeader_1x01_P2.54mm_Vertical, symbol Connector_Generic:Conn_01x01
- added X403: G, Connector_PinHeader_2.54mm:PinHeader_1x01_P2.54mm_Vertical, symbol Connector_Generic:Conn_01x01
- added X404: R, Connector_PinHeader_2.54mm:PinHeader_1x01_P2.54mm_Vertical, symbol Connector_Generic:Conn_01x01
- D0: footprint Package_DIP:DIP-16_W7.62mm_Socket_LongPads -> Package_DIP:DIP-16_W7.62mm_Socket
- R10, R15, R25, R5: footprint Resistor_THT:R_Axial_DIN0207_L6.3mm_D2.5mm_P10.16mm_Horizontal -> Tiny2k_Bauteile:R_Axial_TGL8728_L5.9mm_D2.4mm_P12.50mm_Horizontal
- R20: footprint Resistor_THT:R_Axial_DIN0207_L6.3mm_D2.5mm_P10.16mm_Horizontal -> Resistor_THT:R_Axial_DIN0309_L9.0mm_D3.2mm_P2.54mm_Vertical
- VD400, VD401, VD402, VD403, VD404, VD405: footprint Diode_THT:D_DO-34_SOD68_P2.54mm_Vertical_AnodeUp -> Tiny2k_Bauteile:D_E-Line_P2.5mm_Vertical
- VT400, VT401, VT402, VT403, VT404: footprint Package_TO_SOT_THT:TO-92Flat -> Package_TO_SOT_THT:TO-92_Inline_Wide
Connections:
- net labels removed: B, Blau, G, Grün, R, Rot, S, Sync, V, ~AV~RGB
- wire segments 160 -> 149
- no-connect marks 11 -> 0
Other:
- moved on the sheet: D0B
