File: Erweiterungen/Videoerweiterung/Videoerweiterung_Prozessor.sch (KiCad schematic (older format))
At the start: 39 parts, among them X200 Bus, X201 ~CS2, X202 XTAL, X203 select, X204 ~KEY, X205 BUSY

Commit message: Platine für Videomodul ergänzt
Parts:
- added X206: POWER, Connector_Wire:SolderWire-0.5sqmm_1x02_P4.8mm_D0.9mm_OD2.3mm, symbol Connector_Generic:Conn_01x02
- C202: footprint Capacitor_THT:C_Disc_D5.0mm_W2.5mm_P2.50mm -> Capacitor_THT:C_Disc_D5.0mm_W2.5mm_P5.00mm
- D10, D20, D21: footprint Package_DIP:DIP-16_W7.62mm_Socket_LongPads -> Package_DIP:DIP-16_W7.62mm_Socket
- D13: footprint Package_DIP:DIP-40_W15.24mm_Socket_LongPads -> Package_DIP:DIP-40_W15.24mm_Socket
- D14, D18, D19: footprint Package_DIP:DIP-14_W7.62mm_Socket_LongPads -> Package_DIP:DIP-14_W7.62mm_Socket
- D15, D17, D2, D8: footprint Package_DIP:DIP-20_W7.62mm_Socket_LongPads -> Package_DIP:DIP-20_W7.62mm_Socket
- D5, D6: footprint Package_DIP:DIP-24_W15.24mm_Socket_LongPads -> Package_DIP:DIP-24_W15.24mm_Socket
- R200, R201, R202, R203, R204, R205, R206, R207, R208, R209, R210, R211: footprint Resistor_THT:R_Axial_DIN0207_L6.3mm_D2.5mm_P10.16mm_Horizontal -> Tiny2k_Bauteile:R_Axial_TGL8728_L5.9mm_D2.4mm_P12.50mm_Horizontal
- VD200, VD202: footprint Diode_THT:D_DO-34_SOD68_P2.54mm_Vertical_AnodeUp -> Tiny2k_Bauteile:D_E-Line_P2.5mm_Vertical
- VD201: footprint Diode_THT:D_DO-34_SOD68_P2.54mm_Vertical_AnodeUp -> Diode_THT:D_DO-34_SOD68_P2.54mm_Vertical_KathodeUp
- VT200, VT201: footprint Package_TO_SOT_THT:TO-92Flat -> Package_TO_SOT_THT:TO-92_Inline_Wide
- X202: footprint Connector_PinHeader_2.54mm:PinHeader_1x02_P2.54mm_Vertical -> Connector_PinHeader_2.54mm:PinHeader_1x02_P2.54mm_Horizontal
- X205: footprint Connector_PinHeader_2.54mm:PinHeader_1x01_P2.54mm_Horizontal -> Connector_PinHeader_2.54mm:PinHeader_1x01_P2.54mm_Vertical
Connections:
- net labels added: +5V
- net labels removed: +5P
- no-connect marks 35 -> 31
Other:
- note added: "A4 V/H\nA5 blau\nA6 grün\nA7 rot\n\nL = aktiv\nH = inaktiv"
- note added: "zur\nDaten-\nsteuerung"
- note removed: "A4 V/H\nA5 blau\nA6 grün\nA7 rot"
