File: Erweiterungen/Videoerweiterung/Videoerweiterung_Steuerung_VRAM.sch (KiCad schematic (older format))
At the start: 12 parts, among them X300 8k RAM-Modul, X301 8k RAM-Modul, X302 8k RAM-Modul, X303 8k RAM-Modul

Commit message: Platine für Videomodul ergänzt
Parts:
- D1, D11, D12, D16, D3, D4, D7, D9: footprint Package_DIP:DIP-20_W7.62mm_Socket_LongPads -> Package_DIP:DIP-20_W7.62mm_Socket
Connections:
- net labels added: +5V
- net labels removed: +5P
- wire segments 420 -> 340
Other:
- moved on the sheet: D11B, D12B, D16B, D1B, D3B, D4B, D7B, D9B
