File: Tiny_6k/kicad/Tiny6k_Steuerung_Video-RAM.sch (KiCad schematic (older format))
At the start: 12 parts, among them X300 8k RAM-Modul, X301 8k RAM-Modul, X302 8k RAM-Modul, X303 8k RAM-Modul

Commit message: Übersichtlichkeit erhöht
Other:
- moved on the sheet: D11A, D11B, D12A, D12B, D16A, D16B, D1A, D1B, D3A, D3B, D4A, D4B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

Commit message: Tiny6k_Steuerung_Video-RAM.sch: fix wires
Connections:
- net VBD0: now also D11.8 (A8), D9.13 (B/QB); no longer D11.4 (A4), D9.7 (A/QA)
- net VBD1: now also D11.7 (A7), D9.14 (D/QD); no longer D11.8 (A8), D9.13 (B/QB)
- net VBD2: now also D11.6 (A6), D9.15 (F/QF); no longer D11.3 (A3), D9.6 (C/QC)
- net VBD3: now also D11.5 (A5), D9.16 (H/QH); no longer D11.7 (A7), D9.14 (D/QD)
- net VBD4: now also D11.4 (A4), D9.7 (A/QA); no longer D11.2 (A2), D9.5 (E/QE)
- net VBD5: now also D11.3 (A3), D9.6 (C/QC); no longer D11.6 (A6), D9.15 (F/QF)
- net VBD6: now also D11.2 (A2), D9.5 (E/QE); no longer D11.1 (A1), D9.4 (G/QG)
- net VBD7: now also D11.1 (A1), D9.4 (G/QG); no longer D11.5 (A5), D9.16 (H/QH)
- net VGD0: now also D4.13 (B/QB), D7.8 (A8); no longer D4.7 (A/QA), D7.4 (A4)
- net VGD1: now also D4.14 (D/QD), D7.7 (A7); no longer D4.13 (B/QB), D7.8 (A8)
- net VGD2: now also D4.15 (F/QF), D7.6 (A6); no longer D4.6 (C/QC), D7.3 (A3)
- net VGD3: now also D4.16 (H/QH), D7.5 (A5); no longer D4.14 (D/QD), D7.7 (A7)
- net VGD4: now also D4.7 (A/QA), D7.4 (A4); no longer D4.5 (E/QE), D7.2 (A2)
- net VGD5: now also D4.6 (C/QC), D7.3 (A3); no longer D4.15 (F/QF), D7.6 (A6)
- net VGD6: now also D4.5 (E/QE), D7.2 (A2); no longer D4.4 (G/QG), D7.1 (A1)
- net VGD7: now also D4.4 (G/QG), D7.1 (A1); no longer D4.16 (H/QH), D7.5 (A5)
- net VRD0: now also D1.13 (B/QB), D3.8 (A8); no longer D1.7 (A/QA), D3.4 (A4)
- net VRD1: now also D1.14 (D/QD), D3.7 (A7); no longer D1.13 (B/QB), D3.8 (A8)
- net VRD2: now also D1.15 (F/QF), D3.6 (A6); no longer D1.6 (C/QC), D3.3 (A3)
- net VRD3: now also D1.16 (H/QH), D3.5 (A5); no longer D1.14 (D/QD), D3.7 (A7)
- net VRD4: now also D1.7 (A/QA), D3.4 (A4); no longer D1.5 (E/QE), D3.2 (A2)
- net VRD5: now also D1.6 (C/QC), D3.3 (A3); no longer D1.15 (F/QF), D3.6 (A6)
- net VRD6: now also D1.5 (E/QE), D3.2 (A2); no longer D1.4 (G/QG), D3.1 (A1)
- net VRD7: now also D1.4 (G/QG), D3.1 (A1); no longer D1.16 (H/QH), D3.5 (A5)
- net VVD0: now also D12.13 (B/QB), D16.8 (A8); no longer D12.7 (A/QA), D16.4 (A4)
- net VVD1: now also D12.14 (D/QD), D16.7 (A7); no longer D12.13 (B/QB), D16.8 (A8)
- net VVD2: now also D12.15 (F/QF), D16.6 (A6); no longer D12.6 (C/QC), D16.3 (A3)
- net VVD3: now also D12.16 (H/QH), D16.5 (A5); no longer D12.14 (D/QD), D16.7 (A7)
- net VVD4: now also D12.7 (A/QA), D16.4 (A4); no longer D12.5 (E/QE), D16.2 (A2)
- net VVD5: now also D12.6 (C/QC), D16.3 (A3); no longer D12.15 (F/QF), D16.6 (A6)
- net VVD6: now also D12.5 (E/QE), D16.2 (A2); no longer D12.4 (G/QG), D16.1 (A1)
- net VVD7: now also D12.4 (G/QG), D16.1 (A1); no longer D12.16 (H/QH), D16.5 (A5)
